File: 555_badge.kicad_pcb (KiCad board)
At the start: 2 copper layers, 53.8 x 85.6 mm, 15 parts, among them Q1 2N3904, U1 7555

Commit message: finish board layout
Parts:
- moved R1 8.52 mm to (159.3, 102.9), turned to 270 degrees
- moved R4 7.62 mm to (178.3, 102.9), turned to 270 degrees
- moved R2 3.81 mm to (163.1, 110.5)
- moved Q1 2.54 mm to (166.1, 116.8), turned to 90 degrees
- moved C2 1.44 mm to (175.8, 121.9)
Routing:
- net Net-(D1-Pad1): track 0.00 -> 59.3 mm, vias 0 -> 1
- net Net-(D1-Pad2): track 0.00 -> 54.4 mm
- net VCC: track 0.00 -> 50.7 mm
- net Net-(D2-Pad2): track 0.00 -> 37.9 mm
- net Net-(C1-Pad1): track 0.00 -> 36.9 mm
- net Net-(R3-Pad2): track 0.00 -> 32.7 mm
- net Net-(C2-Pad1): track 0.00 -> 23.7 mm
- net Net-(BAT1-PadPos): track 0.00 -> 15.4 mm
- net Net-(R1-Pad2): track 0.00 -> 11.4 mm
- net Net-(Q1-Pad2): track 0.00 -> 5.19 mm
- added copper zone on B.Cu, net GND
- added copper zone on F.Cu, net GND
Other:
- board text added: "+"
- board text added: "555 Badge"
- board text added: "ON"
- board text added: "m01"
